Commit message: Controller Test: Use UR10 as default robot
Also adjust the tf publisher starting link

File: cartesian_controller_test/robot.urdf.xacro (robot description, xacro)
@@ -2,7 +2,7 @@
 <robot name="robot" xmlns:xacro="http://www.ros.org/wiki/xacro">
         <!-- Includes -->
-        <xacro:include filename="$(find ur_description)/urdf/ur5.urdf.xacro" />
+        <xacro:include filename="$(find ur_description)/urdf/ur10.urdf.xacro" />
         <!-- Create robot instance -->
-        <xacro:ur5_robot prefix="" joint_limited="false"/>
+        <xacro:ur10_robot prefix="" joint_limited="false"/>
         <!-- Connect to world -->
         <link name="world" />
@@ -13,9 +13,10 @@
         </joint>
         <!-- Testing reference frame for tf_publisher_gui -->
+        <!-- Starting frame for tf_publisher_gui -->
         <link name="testing_ref" />
         <joint name="testing_ref_joint" type="fixed">
-                <parent link="world" />
+                <parent link="base_link" />
                 <child link="testing_ref" />
-                <origin xyz="0.386 0.165 0.530" rpy="-3.066 -0.026 -1.426" />
+                <origin xyz="0.543 0.243 0.741" rpy="3.116 -0.077 0.148" />
         </joint>
         <!-- Load control plugin -->

Commit message: Controller Test: Add the sensor link from the test controllers
This sensor link was added to the ur_description urdfs for quick
testing. Now, everybody can test the cartesian_controllers without
modifying anything in the ur_description package.

Also adjust compliance reference for testing.

File: cartesian_controller_test/robot.urdf.xacro (robot description, xacro)
@@ -12,5 +12,11 @@
                 <origin xyz="0.0 0.0 0.0" rpy="0.0 0.0 0.0" />
         </joint>
-        <!-- Testing reference frame for tf_publisher_gui -->
+        <!-- Attach a sensor link -->
+        <link name="sensor_link"/>
+        <joint name="sensor_link_joint" type="fixed">
+                <origin xyz="0 0 0.048" rpy="0 0 ${-pi/2.0}"/>
+                <parent link="tool0"/>
+                <child link="sensor_link"/>
+        </joint>
         <!-- Starting frame for tf_publisher_gui -->
         <link name="testing_ref" />

Commit message: Last changes made by Stefan S for a better controlling

File: cartesian_controller_test/robot.urdf.xacro (robot description, xacro)
@@ -15,5 +15,5 @@
         <link name="sensor_link"/>
         <joint name="sensor_link_joint" type="fixed">
-                <origin xyz="0 0 0.048" rpy="0 0 ${-pi/2.0}"/>
+                <origin xyz="0 0 0.048" rpy="0 0 ${pi/2.0}"/>
                 <parent link="tool0"/>
                 <child link="sensor_link"/>

Commit message: Controller Test: Remove tf-publisher-gui and use interactive control

File: cartesian_controller_test/robot.urdf.xacro (robot description, xacro)
@@ -19,11 +19,4 @@
                 <child link="sensor_link"/>
         </joint>
-        <!-- Starting frame for tf_publisher_gui -->
-        <link name="testing_ref" />
-        <joint name="testing_ref_joint" type="fixed">
-                <parent link="base_link" />
-                <child link="testing_ref" />
-                <origin xyz="0.543 0.243 0.741" rpy="3.116 -0.077 0.148" />
-        </joint>
         <!-- Load control plugin -->
         <!-- This exposes a controller_manager to manage controllers for gazebo -->
