Commit message: Add stiffness and damping parameters to simulation
We can now specify stiffness and damping per joint in the robot
description. This is useful to find stable default controller gains for
MuJoCo.

File: cartesian_controller_simulation/urdf/joint.urdf.xacro (robot description, xacro)
@@ -2,5 +2,5 @@
 <robot xmlns:xacro="http://www.ros.org/wiki/xacro">
         <!-- Individual joint. -->
-        <xacro:macro name="joint_interface" params="name">
+        <xacro:macro name="joint_interface" params="name p d">
                 <joint name="${name}">
                         <command_interface name="position">
@@ -12,4 +12,6 @@
                                 <param name="max">1</param>
                         </command_interface>
+                        <param name="p">${p}</param>
+                        <param name="d">${d}</param>
                         <state_interface name="position"/>
                         <state_interface name="velocity"/>

File: cartesian_controller_simulation/urdf/robot.urdf.xacro (robot description, xacro)
@@ -8,10 +8,10 @@
         <!-- ROS2 control interfaces -->
         <ros2_control name="cartesian_controller_simulation" type="system">
-                <xacro:joint_interface name="joint1" />
-                <xacro:joint_interface name="joint2" />
-                <xacro:joint_interface name="joint3" />
-                <xacro:joint_interface name="joint4" />
-                <xacro:joint_interface name="joint5" />
-                <xacro:joint_interface name="joint6" />
+                <xacro:joint_interface name="joint1" p="80" d="0.4" />
+                <xacro:joint_interface name="joint2" p="80" d="0.4" />
+                <xacro:joint_interface name="joint3" p="80" d="0.4" />
+                <xacro:joint_interface name="joint4" p="80" d="0.4" />
+                <xacro:joint_interface name="joint5" p="80" d="0.4" />
+                <xacro:joint_interface name="joint6" p="10" d="1.0" />
                 <hardware>
                         <plugin>cartesian_controller_simulation/Simulator</plugin>
