Commit message: Add manual test script for joint controller gains
We now have a minimal gui to switch between two hard-coded joint
configurations via a joint trajectory controller.
This is helpful to fine-tune the joint controller gains.

Also lower the robot's link inertias. The previous value of `100` was
unrealistically high. A better next step would be to compute those
values for cylindrical dummies.

File: cartesian_controller_simulation/urdf/robot.urdf.xacro (robot description, xacro)
@@ -8,10 +8,10 @@
         <!-- ROS2 control interfaces -->
         <ros2_control name="cartesian_controller_simulation" type="system">
-                <xacro:joint_interface name="joint1" p="80" d="0.4" />
-                <xacro:joint_interface name="joint2" p="80" d="0.4" />
-                <xacro:joint_interface name="joint3" p="80" d="0.4" />
-                <xacro:joint_interface name="joint4" p="80" d="0.4" />
-                <xacro:joint_interface name="joint5" p="80" d="0.4" />
-                <xacro:joint_interface name="joint6" p="10" d="1.0" />
+                <xacro:joint_interface name="joint1" p="1000" d="0.5" />
+                <xacro:joint_interface name="joint2" p="1000" d="0.5" />
+                <xacro:joint_interface name="joint3" p="500" d="0.5" />
+                <xacro:joint_interface name="joint4" p="100" d="0.5" />
+                <xacro:joint_interface name="joint5" p="10" d="0.5" />
+                <xacro:joint_interface name="joint6" p="10" d="0.5" />
                 <hardware>
                         <plugin>cartesian_controller_simulation/Simulator</plugin>
@@ -65,5 +65,5 @@
                         <origin xyz="0 0 ${joint_length / 2.0}" rpy="0 0 0"/>
                         <mass value="1"/>
-                        <inertia ixx="100"  ixy="0"  ixz="0" iyy="100" iyz="0" izz="100" />
+                        <inertia ixx="1.0"  ixy="0"  ixz="0" iyy="1.0" iyz="0" izz="1.0" />
                 </inertial>
                 <visual name="base">
@@ -86,5 +86,5 @@
                         <origin xyz="0 0 ${link1_length / 2.0}" rpy="0 0 0"/>
                         <mass value="1"/>
-                        <inertia ixx="100"  ixy="0"  ixz="0" iyy="100" iyz="0" izz="100" />
+                        <inertia ixx="1.0"  ixy="0"  ixz="0" iyy="1.0" iyz="0" izz="1.0" />
                 </inertial>
                 <visual name="joint1">
@@ -119,5 +119,5 @@
                         <origin xyz="0 0 ${link2_length / 2.0}" rpy="0 0 0"/>
                         <mass value="1"/>
-                        <inertia ixx="100"  ixy="0"  ixz="0" iyy="100" iyz="0" izz="100" />
+                        <inertia ixx="1.0"  ixy="0"  ixz="0" iyy="1.0" iyz="0" izz="1.0" />
                 </inertial>
                 <visual name="joint2">
@@ -152,5 +152,5 @@
                         <origin xyz="0 0 ${link3_length / 2.0}" rpy="0 0 0"/>
                         <mass value="1"/>
-                        <inertia ixx="100"  ixy="0"  ixz="0" iyy="100" iyz="0" izz="100" />
+                        <inertia ixx="1.0"  ixy="0"  ixz="0" iyy="1.0" iyz="0" izz="1.0" />
                 </inertial>
                 <visual name="joint3">
@@ -185,5 +185,5 @@
                         <origin xyz="0 0 ${link4_length / 2.0}" rpy="0 0 0"/>
                         <mass value="1"/>
-                        <inertia ixx="100"  ixy="0"  ixz="0" iyy="100" iyz="0" izz="100" />
+                        <inertia ixx="1.0"  ixy="0"  ixz="0" iyy="1.0" iyz="0" izz="1.0" />
                 </inertial>
                 <visual name="joint4">
@@ -218,5 +218,5 @@
                         <origin xyz="0 0 ${link5_length / 2.0}" rpy="0 0 0"/>
                         <mass value="1"/>
-                        <inertia ixx="100"  ixy="0"  ixz="0" iyy="100" iyz="0" izz="100" />
+                        <inertia ixx="1.0"  ixy="0"  ixz="0" iyy="1.0" iyz="0" izz="1.0" />
                 </inertial>
                 <visual name="joint5">
@@ -251,5 +251,5 @@
                         <origin xyz="0 0 ${link6_length / 2.0}" rpy="0 0 0"/>
                         <mass value="1"/>
-                        <inertia ixx="100"  ixy="0"  ixz="0" iyy="100" iyz="0" izz="100" />
+                        <inertia ixx="1.0"  ixy="0"  ixz="0" iyy="1.0" iyz="0" izz="1.0" />
                 </inertial>
                 <visual name="joint6">

Commit message: Add additional urdf links for integration tests
We'll need them to specify invalid kinematic chains.

File: cartesian_controller_simulation/urdf/robot.urdf.xacro (robot description, xacro)
@@ -61,4 +61,11 @@
                 <color rgba="0.988 0.580 0.450 1.0"/>
         </material>
+        <!-- Connect to world -->
+        <link name="world" />
+        <joint name="world_joint" type="fixed">
+                <parent link="world" />
+                <child link = "base_link" />
+                <origin xyz="0.0 0.0 0.0" rpy="0.0 0.0 0.0" />
+        </joint>
         <link name="base_link" >
                 <inertial>
@@ -267,18 +274,4 @@
                 </visual>
         </link>
-        <joint name="tool0_joint" type="fixed">
-                <origin xyz="0 0 ${link6_length / 2.0}" rpy="0 0 0"/>
-                <parent link="sensor_link"/>
-                <child link="tool0"/>
-        </joint>
-        <link name="tool0">
-                <visual>
-                        <origin xyz="0 0 0" rpy="0 0 0" />
-                        <geometry>
-                                <sphere radius="${link_radius}"/>
-                        </geometry>
-                        <material name="tip"/>
-                </visual>
-        </link>
         <!-- Attach a sensor link -->
         <joint name="sensor_link_joint" type="fixed">
@@ -288,10 +281,31 @@
         </joint>
         <link name="sensor_link"/>
-        <!-- Connect to world -->
-        <link name="world" />
-        <joint name="world_joint" type="fixed">
-                <parent link="world" />
-                <child link = "base_link" />
-                <origin xyz="0.0 0.0 0.0" rpy="0.0 0.0 0.0" />
-        </joint>
+        <!-- The default end-effector -->
+        <joint name="tool0_joint" type="fixed">
+                <origin xyz="0 0 ${link6_length / 2.0}" rpy="0 0 0"/>
+                <parent link="sensor_link"/>
+                <child link="tool0"/>
+        </joint>
+        <link name="tool0">
+                <visual>
+                        <origin xyz="0 0 0" rpy="0 0 0" />
+                        <geometry>
+                                <sphere radius="${link_radius}"/>
+                        </geometry>
+                        <material name="tip"/>
+                </visual>
+        </link>
+        <!-- Additional links for integration tests. -->
+        <joint name="invalid_sensor_link_joint" type="fixed">
+                <origin xyz="0 ${link6_length / 2.0} 0" rpy="${-pi / 2.0} 0 0"/>
+                <parent link="link6"/>
+                <child link="invalid_sensor_link"/>
+        </joint>
+        <link name="invalid_sensor_link"/>
+        <joint name="invalid_compliance_link_joint" type="fixed">
+                <origin xyz="0 0 0" rpy="0 0 0"/>
+                <parent link="sensor_link"/>
+                <child link="invalid_compliance_link"/>
+        </joint>
+        <link name="invalid_compliance_link"/>
 </robot>
