Commit message: Examples: Adjust joint positions
The poses of the link TFs are now more consistent.

File: cartesian_controller_examples/urdf/robot.urdf.xacro (robot description, xacro)
@@ -15,5 +15,5 @@
         <xacro:property name="link4_length" value="0.15" />
         <xacro:property name="link5_length" value="0.10" />
-        <xacro:property name="link6_length" value="0.1" />
+        <xacro:property name="link6_length" value="0.05" />
         <!-- colors -->
         <material name="grey">
@@ -32,5 +32,5 @@
                 <parent link="base_link" />
                 <child link = "link1" />
-                <origin xyz="0.0 0.0 ${joint_length}" rpy="0.0 0.0 0.0" />
+                <origin xyz="0.0 0.0 ${3.0 / 2.0 * joint_length}" rpy="0.0 0.0 0.0" />
                 <axis xyz="0 0 1" />
                 <limit lower="${-2.0 * pi}" upper="${2.0 * pi}" effort="1.0" velocity="10.0"/>
@@ -38,5 +38,5 @@
         <link name="link1">
                 <visual name="joint1">
-                        <origin xyz="0 0 ${joint_length / 2.0}" rpy="0 0 0" />
+                        <origin xyz="0 0 0" rpy="0 0 0" />
                         <geometry>
                                 <cylinder length="${joint_length}" radius="${joint_radius}"/>
@@ -122,5 +122,5 @@
                 <parent link="link3" />
                 <child link = "link4" />
-                <origin xyz="0.0 0.0 ${link3_length}" rpy="0.0 ${pi / 2.0} 0.0" />
+                <origin xyz="0.0 ${joint_length} ${link3_length}" rpy="0.0 ${pi / 2.0} 0.0" />
                 <axis xyz="0 1 0" />
                 <limit lower="${-2.0 * pi}" upper="${2.0 * pi}" effort="1.0" velocity="10.0"/>
@@ -128,5 +128,5 @@
         <link name="link4">
                 <visual name="joint4">
-                        <origin xyz="0 ${joint_length} 0" rpy="${pi / 2.0} 0 0" />
+                        <origin xyz="0 0 0" rpy="${pi / 2.0} 0 0" />
                         <geometry>
                                 <cylinder length="${joint_length}" radius="${joint_radius}"/>
@@ -152,5 +152,5 @@
                 <parent link="link4" />
                 <child link = "link5" />
-                <origin xyz="0.0 ${link4_length} 0.0" rpy="0.0 0.0 0.0" />
+                <origin xyz="0.0 ${link4_length} ${joint_length}" rpy="0.0 0.0 0.0" />
                 <axis xyz="0 0 1" />
                 <limit lower="${-2.0 * pi}" upper="${2.0 * pi}" effort="1.0" velocity="10.0"/>
@@ -158,5 +158,5 @@
         <link name="link5">
                 <visual name="joint5">
-                        <origin xyz="0 0 ${joint_length}" rpy="0 0 0" />
+                        <origin xyz="0 0 0" rpy="0 0 0" />
                         <geometry>
                                 <cylinder length="${joint_length}" radius="${joint_radius}"/>
@@ -182,5 +182,5 @@
                 <parent link="link5" />
                 <child link = "link6" />
-                <origin xyz="0.0 0.0 ${link5_length}" rpy="0.0 0.0 0.0" />
+                <origin xyz="0.0 ${joint_length} ${link5_length}" rpy="0.0 0.0 0.0" />
                 <axis xyz="0 1 0" />
                 <limit lower="${-2.0 * pi}" upper="${2.0 * pi}" effort="1.0" velocity="10.0"/>
@@ -188,5 +188,5 @@
         <link name="link6">
                 <visual name="joint6">
-                        <origin xyz="0 ${joint_length} 0" rpy="${pi / 2.0} 0 0" />
+                        <origin xyz="0 0 0" rpy="${pi / 2.0} 0 0" />
                         <geometry>
                                 <cylinder length="${joint_length}" radius="${joint_radius}"/>
@@ -216,4 +216,11 @@
                 </visual>
         </link>
+        <!-- Attach a sensor link -->
+        <joint name="sensor_link_joint" type="fixed">
+                <origin xyz="0 ${link6_length / 2.0} 0" rpy="${-pi / 2.0} 0 ${pi / 2.0}"/>
+                <parent link="link6"/>
+                <child link="sensor_link"/>
+        </joint>
+        <link name="sensor_link"/>
         <!-- Connect to world -->
         <link name="world" />
@@ -223,10 +230,3 @@
                 <origin xyz="0.0 0.0 0.0" rpy="0.0 0.0 0.0" />
         </joint>
-        <!-- Attach a sensor link -->
-        <link name="sensor_link"/>
-        <joint name="sensor_link_joint" type="fixed">
-                <origin xyz="0 0 0.048" rpy="0 0 ${pi/2.0}"/>
-                <parent link="tool0"/>
-                <child link="sensor_link"/>
-        </joint>
 </robot>

Commit message: update urdf issue#32 suggests

File: cartesian_controller_examples/urdf/robot.urdf.xacro (robot description, xacro)
@@ -203,6 +203,6 @@
         </link>
         <joint name="tool0_joint" type="fixed">
-                <origin xyz="0 ${link6_length} 0" rpy="${-pi / 2.0} 0 0"/>
-                <parent link="link6"/>
+                <origin xyz="${link6_length / 2.0} 0 0" rpy="0 ${pi / 2.0} 0"/>
+                <parent link="sensor_link"/>
                 <child link="tool0"/>
         </joint>

Commit message: align z-axis in sensor_link with one in tool0

File: cartesian_controller_examples/urdf/robot.urdf.xacro (robot description, xacro)
@@ -203,5 +203,5 @@
         </link>
         <joint name="tool0_joint" type="fixed">
-                <origin xyz="${link6_length / 2.0} 0 0" rpy="0 ${pi / 2.0} 0"/>
+                <origin xyz="0 0 ${link6_length / 2.0}" rpy="0 0 0"/>
                 <parent link="sensor_link"/>
                 <child link="tool0"/>
@@ -218,5 +218,5 @@
         <!-- Attach a sensor link -->
         <joint name="sensor_link_joint" type="fixed">
-                <origin xyz="0 ${link6_length / 2.0} 0" rpy="${-pi / 2.0} 0 ${pi / 2.0}"/>
+                <origin xyz="0 ${link6_length / 2.0} 0" rpy="${-pi / 2.0} 0 0"/>
                 <parent link="link6"/>
                 <child link="sensor_link"/>

Commit message: update robot.urdf.xacro urdf like mentioned at issue #32 (#48)
* update urdf issue#32 suggests

* align z-axis in sensor_link with one in tool0

File: cartesian_controller_examples/urdf/robot.urdf.xacro (robot description, xacro)
@@ -203,6 +203,6 @@
         </link>
         <joint name="tool0_joint" type="fixed">
-                <origin xyz="0 ${link6_length} 0" rpy="${-pi / 2.0} 0 0"/>
-                <parent link="link6"/>
+                <origin xyz="0 0 ${link6_length / 2.0}" rpy="0 0 0"/>
+                <parent link="sensor_link"/>
                 <child link="tool0"/>
         </joint>
@@ -218,5 +218,5 @@
         <!-- Attach a sensor link -->
         <joint name="sensor_link_joint" type="fixed">
-                <origin xyz="0 ${link6_length / 2.0} 0" rpy="${-pi / 2.0} 0 ${pi / 2.0}"/>
+                <origin xyz="0 ${link6_length / 2.0} 0" rpy="${-pi / 2.0} 0 0"/>
                 <parent link="link6"/>
                 <child link="sensor_link"/>
